File: dcapacitors.kicad_sch (KiCad schematic)
At the start: 55 parts

Commit message: Add LCSC Basic/Extended part numbers for JLC-placed passives and ferrite beads
Parts:
- C24: LCSC Part (none) -> C49066
- C25, C26, C27, C28, C29: LCSC Part (none) -> C2932477
- C30, C31, C32, C33, C34, C35, C36, C37, C38, C39, C40, C41, C42, C43, C44, C45, C46: LCSC Part (none) -> C98195
- C47, C48, C49, C50, C51, C52, C53, C54, C55, C56, C57, C58, C59, C60, C61, C62, C63, C64, C65, C66, C67, C68, C69, C70, C71, C72, C73, C74, C75, C76, C77, C78: LCSC Part (none) -> C1623
