File: ethernet1g.kicad_sch (KiCad schematic)
At the start: 32 parts, among them J3 HR911130C, U8 RTL8211E-VB-CG, Y3 OT322525MJBA4SL

Commit message: Add LCSC Basic/Extended part numbers for JLC-placed passives and ferrite beads
Parts:
- C100, C101, C102, C91, C92, C93, C94, C95, C96, C97, C98, C99: LCSC Part (none) -> C14663
- C103, C104, C105: LCSC Part (none) -> C98195
- FB4, FB5: LCSC Part (none) -> C19330
- R29: LCSC Part (none) -> C2930072
Changed lines of the file:
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@@
 			)
 		)
+		(property "LCSC Part" "C14663"
+			(at 0 0 0)
+			(hide yes)
+			(show_name no)
+			(do_not_autoplace no)
+			(effects
+				(font
+					(size 1.27 1.27)
+				)
+			)
+		)
 		(property "Datasheet" ""
 			(at 292.1 86.36 0)
@@
 			)
 		)
+		(property "LCSC Part" "C14663"
+			(at 0 0 0)
+			(hide yes)
+			(show_name no)
+			(do_not_autoplace no)
+			(effects
+				(font
+					(size 1.27 1.27)
+				)
+			)
+		)
 		(property "Datasheet" ""
 			(at 293.37 127 0)
@@
 			)
 		)
+		(property "LCSC Part" "C98195"
+			(at 0 0 0)
+			(hide yes)
+			(show_name no)
+			(do_not_autoplace no)
+			(effects
+				(font
+					(size 1.27 1.27)
+				)
+			)
+		)
 		(property "Datasheet" ""
 			(at 375.92 125.73 0)
@@
 			)
 		)
+		(property "LCSC Part" "C98195"
+			(at 0 0 0)
+			(hide yes)
+			(show_name no)
+			(do_not_autoplace no)
+			(effects
+				(font
+					(size 1.27 1.27)
+				)
+			)
+		)
 		(property "Datasheet" ""
 			(at 344.17 127 0)
@@
 			)
 		)
+		(property "LCSC Part" "C19330"
+			(at 0 0 0)
+			(hide yes)
+			(show_name no)
+			(do_not_autoplace no)
+			(effects
+				(font
+					(size 1.27 1.27)
+				)
+			)
+		)
 		(property "Datasheet" ""
 			(at 298.45 35.56 0)
@@
 			)
 		)
+		(property "LCSC Part" "C19330"
+			(at 0 0 0)
+			(hide yes)
+			(show_name no)
+			(do_not_autoplace no)
+			(effects
+				(font
+					(size 1.27 1.27)
+				)
+			)
+		)
 		(property "Datasheet" ""
 			(at 306.07 35.56 0)
@@
 			)
 		)
+		(property "LCSC Part" "C14663"
+			(at 0 0 0)
+			(hide yes)
+			(show_name no)
+			(do_not_autoplace no)
+			(effects
+				(font
+					(size 1.27 1.27)
+				)
+			)
+		)
 		(property "Datasheet" ""
 			(at 307.34 127 0)
@@
 			)
 		)
+		(property "LCSC Part" "C14663"
+			(at 0 0 0)
+			(hide yes)
+			(show_name no)
+			(do_not_autoplace no)
+			(effects
+				(font
+					(size 1.27 1.27)
+				)
+			)
+		)
 		(property "Datasheet" ""
 			(at 368.3 86.36 0)
@@
 			)
 		)
+		(property "LCSC Part" "C14663"
+			(at 0 0 0)
+			(hide yes)
+			(show_name no)
+			(do_not_autoplace no)
+			(effects
+				(font
+					(size 1.27 1.27)
+				)
+			)
+		)
 		(property "Datasheet" ""
 			(at 317.5 86.36 0)
@@
 			)
 		)
+		(property "LCSC Part" "C14663"
+			(at 0 0 0)
+			(hide yes)
+			(show_name no)
+			(do_not_autoplace no)
+			(effects
+				(font
+					(size 1.27 1.27)
+				)
+			)
+		)
 		(property "Datasheet" ""
 			(at 355.6 86.36 0)
@@
 			)
 		)
+		(property "LCSC Part" "C14663"
+			(at 0 0 0)
+			(hide yes)
+			(show_name no)
+			(do_not_autoplace no)
+			(effects
+				(font
+					(size 1.27 1.27)
+				)
+			)
+		)
 		(property "Datasheet" ""
 			(at 332.74 127 0)
@@
 			)
 		)
+		(property "LCSC Part" "C14663"
+			(at 0 0 0)
+			(hide yes)
+			(show_name no)
+			(do_not_autoplace no)
+			(effects
+				(font
+					(size 1.27 1.27)
+				)
+			)
+		)
 		(property "Datasheet" ""
 			(at 342.9 86.36 0)
@@
 			)
 		)
+		(property "LCSC Part" "C14663"
+			(at 0 0 0)
+			(hide yes)
+			(show_name no)
+			(do_not_autoplace no)
+			(effects
+				(font
+					(size 1.27 1.27)
+				)
+			)
+		)
 		(property "Datasheet" ""
 			(at 389.89 34.29 0)
@@
 			)
 		)
+		(property "LCSC Part" "C2930072"
+			(at 0 0 0)
+			(hide yes)
+			(show_name no)
+			(do_not_autoplace no)
+			(effects
+				(font
+					(size 1.27 1.27)
+				)
+			)
+		)
 		(property "Datasheet" ""
 			(at 100.33 132.08 0)
@@
 			)
 		)
+		(property "LCSC Part" "C14663"
+			(at 0 0 0)
+			(hide yes)
+			(show_name no)
+			(do_not_autoplace no)
+			(effects
+				(font
+					(size 1.27 1.27)
+				)
+			)
+		)
 		(property "Datasheet" ""
 			(at 330.2 86.36 0)
@@
 			)
 		)
+		(property "LCSC Part" "C14663"
+			(at 0 0 0)
+			(hide yes)
+			(show_name no)
+			(do_not_autoplace no)
+			(effects
+				(font
+					(size 1.27 1.27)
+				)
+			)
+		)
 		(property "Datasheet" ""
 			(at 304.8 86.36 0)
@@
 			)
 		)
+		(property "LCSC Part" "C98195"
+			(at 0 0 0)
+			(hide yes)
+			(show_name no)
+			(do_not_autoplace no)
+			(effects
+				(font
+					(size 1.27 1.27)
+				)
+			)
+		)
 		(property "Datasheet" ""
 			(at 388.62 125.73 0)
@@
 			(hide yes)
 			(show_name no)
+			(do_not_autoplace no)
+			(effects
+				(font
+					(size 1.27 1.27)
+				)
+			)
+		)
+		(property "LCSC Part" "C14663"
+			(at 0 0 0)
+			(hide yes)
+			(show_name no)

Commit message: Add optional ESP32-C3 WiFi sheet, convert hand-solder parts to through-hole
- New wifi sheet: ESP32-C3-MINI-1 module on SPI to spare FPGA bank 34, with EN/boot-strap networks, 3V3 bypass/bulk caps and a UART debug header
- Replace SMD hand-solder resistors, LEDs, zener, fuse and ceramic caps with THT equivalents; bulk 10uF/22uF caps become polarized electrolytics
- Fill in LCSC part numbers for the new parts and regenerate BOM and ERC report
Parts:
- C106: footprint Capacitor_SMD:C_0603_1608Metric_Pad1.08x0.95mm_HandSolder -> Capacitor_THT:C_Disc_D3.0mm_W2.0mm_P2.50mm; LCSC Part (none) -> C5632430
- R30, R31, R32, R33, R34, R35, R36, R37, R38, R39: footprint Resistor_SMD:R_0603_1608Metric_Pad0.98x0.95mm_HandSolder -> Resistor_THT:R_Axial_DIN0207_L6.3mm_D2.5mm_P10.16mm_Horizontal

Commit message: Pre-routing checkpoint: zone pours, net labels, decoupling on bottom, R51 1k
- GND pours on F.Cu, In1.Cu, In4.Cu, B.Cu; In3.Cu power pours for 1V0, 1V8,
  5V_LC, MGTAVCC, MGTAVTT, 3V3 (3V3 lowest priority)
- Local labels on previously unnamed power nets
- FPGA decoupling moved to B.Cu under/around U6
- R51 (PUDC_B pull-up) 4.7k -> 1k per UG470
- Silkscreen cleanup
Connections:
- net PHY_RSET: now reaches R29.1, U8.39 (RSET)
Changed lines of the file:
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@@
+		)
+	)
+	(label "PHY_RSET"
+		(at 100.33 128.27 90)
+		(effects
+			(font
+				(size 1.27 1.27)
+			)
+			(justify left bottom)
 		)
 	)
