File: iobreakout.kicad_sch (KiCad schematic)
At the start: 14 parts, among them J5 Conn_02x10_Odd_Even, SW2 SW_Push, SW3 SW_Push

Commit message: Add optional ESP32-C3 WiFi sheet, convert hand-solder parts to through-hole
- New wifi sheet: ESP32-C3-MINI-1 module on SPI to spare FPGA bank 34, with EN/boot-strap networks, 3V3 bypass/bulk caps and a UART debug header
- Replace SMD hand-solder resistors, LEDs, zener, fuse and ceramic caps with THT equivalents; bulk 10uF/22uF caps become polarized electrolytics
- Fill in LCSC part numbers for the new parts and regenerate BOM and ERC report
Parts:
- D3, D4, D5, D6: footprint LED_SMD:LED_0603_1608Metric_Pad1.05x0.95mm_HandSolder -> LED_THT:LED_D3.0mm
- R45, R46, R47, R48, R49, R50, R51: footprint Resistor_SMD:R_0603_1608Metric_Pad0.98x0.95mm_HandSolder -> Resistor_THT:R_Axial_DIN0207_L6.3mm_D2.5mm_P10.16mm_Horizontal
Changed lines of the file:
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@@
 			)
 		)
-		(property "Footprint" "LED_SMD:LED_0603_1608Metric_Pad1.05x0.95mm_HandSolder"
+		(property "Footprint" "LED_THT:LED_D3.0mm"
 			(at 143.51 67.31 0)
 			(hide yes)
@@
 			)
 		)
-		(property "Footprint" "Resistor_SMD:R_0603_1608Metric_Pad0.98x0.95mm_HandSolder"
+		(property "Footprint" "Resistor_THT:R_Axial_DIN0207_L6.3mm_D2.5mm_P10.16mm_Horizontal"
 			(at 134.62 55.118 90)
 			(hide yes)
@@
 			)
 		)
-		(property "Footprint" "LED_SMD:LED_0603_1608Metric_Pad1.05x0.95mm_HandSolder"
+		(property "Footprint" "LED_THT:LED_D3.0mm"
 			(at 143.51 53.34 0)
 			(hide yes)
@@
 			)
 		)
-		(property "Footprint" "LED_SMD:LED_0603_1608Metric_Pad1.05x0.95mm_HandSolder"
+		(property "Footprint" "LED_THT:LED_D3.0mm"
 			(at 143.51 26.67 0)
 			(hide yes)
@@
 			)
 		)
-		(property "Footprint" "Resistor_SMD:R_0603_1608Metric_Pad0.98x0.95mm_HandSolder"
+		(property "Footprint" "Resistor_THT:R_Axial_DIN0207_L6.3mm_D2.5mm_P10.16mm_Horizontal"
 			(at 134.62 69.088 90)
 			(hide yes)
@@
 			)
 		)
-		(property "Footprint" "LED_SMD:LED_0603_1608Metric_Pad1.05x0.95mm_HandSolder"
+		(property "Footprint" "LED_THT:LED_D3.0mm"
 			(at 143.51 39.37 0)
 			(hide yes)
@@
 			)
 		)
-		(property "Footprint" "Resistor_SMD:R_0603_1608Metric_Pad0.98x0.95mm_HandSolder"
+		(property "Footprint" "Resistor_THT:R_Axial_DIN0207_L6.3mm_D2.5mm_P10.16mm_Horizontal"
 			(at 40.64 25.908 90)
 			(hide yes)
@@
 			)
 		)
-		(property "Footprint" "Resistor_SMD:R_0603_1608Metric_Pad0.98x0.95mm_HandSolder"
+		(property "Footprint" "Resistor_THT:R_Axial_DIN0207_L6.3mm_D2.5mm_P10.16mm_Horizontal"
 			(at 134.62 28.448 90)
 			(hide yes)
@@
 			)
 		)
-		(property "Footprint" "Resistor_SMD:R_0603_1608Metric_Pad0.98x0.95mm_HandSolder"
+		(property "Footprint" "Resistor_THT:R_Axial_DIN0207_L6.3mm_D2.5mm_P10.16mm_Horizontal"
 			(at 87.63 50.038 90)
 			(hide yes)
@@
 			)
 		)
-		(property "Footprint" "Resistor_SMD:R_0603_1608Metric_Pad0.98x0.95mm_HandSolder"
+		(property "Footprint" "Resistor_THT:R_Axial_DIN0207_L6.3mm_D2.5mm_P10.16mm_Horizontal"
 			(at 134.62 41.148 90)
 			(hide yes)
@@
 			)
 		)
-		(property "Footprint" "Resistor_SMD:R_0603_1608Metric_Pad0.98x0.95mm_HandSolder"
+		(property "Footprint" "Resistor_THT:R_Axial_DIN0207_L6.3mm_D2.5mm_P10.16mm_Horizontal"
 			(at 40.64 51.308 90)
 			(hide yes)

Commit message: Pre-routing checkpoint: zone pours, net labels, decoupling on bottom, R51 1k
- GND pours on F.Cu, In1.Cu, In4.Cu, B.Cu; In3.Cu power pours for 1V0, 1V8,
  5V_LC, MGTAVCC, MGTAVTT, 3V3 (3V3 lowest priority)
- Local labels on previously unnamed power nets
- FPGA decoupling moved to B.Cu under/around U6
- R51 (PUDC_B pull-up) 4.7k -> 1k per UG470
- Silkscreen cleanup
Parts:
- R51: value 4.7k -> 1k
Changed lines of the file:
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@@
 		(fields_autoplaced yes)
 		(property "Reference" "R51"
-			(at 86.3599 45.72 0)
+			(at 87.63 41.91 90)
 			(show_name no)
 			(do_not_autoplace no)
@@
 					(size 1.27 1.27)
 				)
-				(justify left)
 			)
 		)
-		(property "Value" "4.7k"
-			(at 88.8999 45.72 0)
+		(property "Value" "1k"
+			(at 87.63 44.45 90)
 			(show_name no)
 			(do_not_autoplace no)
@@
 					(size 1.27 1.27)
 				)
-				(justify left)
 			)
 		)
