File: powerrails.kicad_sch (KiCad schematic)
At the start: 45 parts, among them U1 TPS62130A, U2 TPS62130A, U3 TPS62130A, U4 TPS62130A

Commit message: Add optional ESP32-C3 WiFi sheet, convert hand-solder parts to through-hole
- New wifi sheet: ESP32-C3-MINI-1 module on SPI to spare FPGA bank 34, with EN/boot-strap networks, 3V3 bypass/bulk caps and a UART debug header
- Replace SMD hand-solder resistors, LEDs, zener, fuse and ceramic caps with THT equivalents; bulk 10uF/22uF caps become polarized electrolytics
- Fill in LCSC part numbers for the new parts and regenerate BOM and ERC report
Parts:
- C1, C2, C3, C4: footprint Capacitor_SMD:C_1210_3225Metric_Pad1.33x2.70mm_HandSolder -> Capacitor_THT:CP_Radial_D5.0mm_P2.00mm; symbol Device:C -> Device:C_Polarized; LCSC Part (none) -> C47344176
- C10, C11, C12, C9: footprint Capacitor_SMD:C_0603_1608Metric_Pad1.08x0.95mm_HandSolder -> Capacitor_THT:C_Disc_D3.0mm_W2.0mm_P2.50mm; LCSC Part (none) -> C511575
- C13, C14, C15, C16, C17, C18, C19, C20: footprint Capacitor_SMD:C_0805_2012Metric_Pad1.18x1.45mm_HandSolder -> Capacitor_THT:CP_Radial_D6.3mm_P2.50mm; symbol Device:C -> Device:C_Polarized; LCSC Part (none) -> C2835673
- C5, C6, C7, C8: footprint Capacitor_SMD:C_0603_1608Metric_Pad1.08x0.95mm_HandSolder -> Capacitor_THT:C_Disc_D3.0mm_W2.0mm_P2.50mm; LCSC Part (none) -> C5632430
- D1: footprint LED_SMD:LED_0603_1608Metric_Pad1.05x0.95mm_HandSolder -> LED_THT:LED_D3.0mm
- R1, R10, R11, R12, R2, R3, R4, R5, R6, R7, R8, R9: footprint Resistor_SMD:R_0603_1608Metric_Pad0.98x0.95mm_HandSolder -> Resistor_THT:R_Axial_DIN0207_L6.3mm_D2.5mm_P10.16mm_Horizontal

Commit message: Pre-routing checkpoint: zone pours, net labels, decoupling on bottom, R51 1k
- GND pours on F.Cu, In1.Cu, In4.Cu, B.Cu; In3.Cu power pours for 1V0, 1V8,
  5V_LC, MGTAVCC, MGTAVTT, 3V3 (3V3 lowest priority)
- Local labels on previously unnamed power nets
- FPGA decoupling moved to B.Cu under/around U6
- R51 (PUDC_B pull-up) 4.7k -> 1k per UG470
- Silkscreen cleanup
Connections:
- net FB_1V2: now reaches R5.2, R6.1, U3.5 (FB)
- net SS_1V8: now reaches C10.1, U2.9 (SS/TR)
- net FB_3V3: now reaches R7.2, R8.1, U4.5 (FB)
- net SW_1V2: now reaches L3.2, U3.1 (SW), U3.2 (SW), U3.3 (SW)
- net FB_1V0: now reaches R1.2, R2.1, U1.5 (FB)
- net SW_3V3: now reaches L4.2, U4.1 (SW), U4.2 (SW), U4.3 (SW)
- net FB_1V8: now reaches R3.2, R4.1, U2.5 (FB)
- net SW_1V0: now reaches L1.2, U1.1 (SW), U1.2 (SW), U1.3 (SW)
- net SS_1V0: now reaches C9.1, U1.9 (SS/TR)
- net SS_3V3: now reaches C12.1, U4.9 (SS/TR)
- net SW_1V8: now reaches L2.2, U2.1 (SW), U2.2 (SW), U2.3 (SW)
- net SS_1V2: now reaches C11.1, U3.9 (SS/TR)
Changed lines of the file:
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@@
+		)
+	)
+	(label "FB_3V3"
+		(at 257.81 73.66 270)
+		(effects
+			(font
+				(size 1.27 1.27)
+			)
+			(justify right bottom)
+		)
+	)
+	(label "SS_1V0"
+		(at 25.4 71.12 90)
+		(effects
+			(font
+				(size 1.27 1.27)
+			)
+			(justify left bottom)
+		)
+	)
+	(label "FB_1V2"
+		(at 194.31 73.66 270)
+		(effects
+			(font
+				(size 1.27 1.27)
+			)
+			(justify right bottom)
+		)
+	)
+	(label "FB_1V8"
+		(at 129.54 74.93 270)
+		(effects
+			(font
+				(size 1.27 1.27)
+			)
+			(justify right bottom)
+		)
+	)
+	(label "SW_1V0"
+		(at 57.15 63.5 270)
+		(effects
+			(font
+				(size 1.27 1.27)
+			)
+			(justify right bottom)
+		)
+	)
+	(label "FB_1V0"
+		(at 62.23 73.66 270)
+		(effects
+			(font
+				(size 1.27 1.27)
+			)
+			(justify right bottom)
+		)
+	)
+	(label "SS_1V8"
+		(at 91.44 72.39 90)
+		(effects
+			(font
+				(size 1.27 1.27)
+			)
+			(justify left bottom)
+		)
+	)
+	(label "SW_1V2"
+		(at 187.96 62.23 270)
+		(effects
+			(font
+				(size 1.27 1.27)
+			)
+			(justify right bottom)
+		)
+	)
+	(label "SW_3V3"
+		(at 251.46 60.96 270)
+		(effects
+			(font
+				(size 1.27 1.27)
+			)
+			(justify right bottom)
+		)
+	)
+	(label "SW_1V8"
+		(at 124.46 63.5 270)
+		(effects
+			(font
+				(size 1.27 1.27)
+			)
+			(justify right bottom)
+		)
+	)
+	(label "SS_1V2"
+		(at 154.94 73.66 90)
+		(effects
+			(font
+				(size 1.27 1.27)
+			)
+			(justify left bottom)
+		)
+	)
+	(label "SS_3V3"
+		(at 218.44 72.39 90)
+		(effects
+			(font
+				(size 1.27 1.27)
+			)
+			(justify left bottom)
 		)
 	)

Commit message: Routing in progress: In3 power pours, DONE LED, DRC cleanup
- Add CFG_DONE 330R pull-up (R52) and DONE LED (D7, R53) per UG470
- Redraw In3.Cu pours to sit under their U6 balls (1V0 core, 1V8 strip,
  MGTAVCC, MGTAVTT); trim 5V_LC strip to y=50; zone clearance 0.2mm
- Remove 3V3/5V_LC traces from In4.Cu GND plane
- Custom rules: U6 BGA escape, solid GND on regulators/tight caps,
  1-spoke thermals on J4 and C22
- Fix clearance violations, remove dangling vias and stubs
- Remaining: GND pours split on In1.Cu/B.Cu by signal traces on In1.Cu
Connections:
- net FB_1V0: no longer names the net of R1.2, R2.1, U1.5 (FB)
- net SS_1V0: no longer names the net of C9.1, U1.9 (SS/TR)
- net SW_1V0: no longer names the net of L1.2, U1.1 (SW), U1.2 (SW), U1.3 (SW)
Changed lines of the file:
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@@
-		)
-	)
-	(label "SS_1V0"
-		(at 25.4 71.12 90)
-		(effects
-			(font
-				(size 1.27 1.27)
-			)
-			(justify left bottom)
 		)
 	)
@@
 		(effects
 			(font
-				(size 1.27 1.27)
-			)
-			(justify right bottom)
-		)
-	)
-	(label "SW_1V0"
-		(at 57.15 63.5 270)
-		(effects
-			(font
-				(size 1.27 1.27)
-			)
-			(justify right bottom)
-		)
-	)
-	(label "FB_1V0"
-		(at 62.23 73.66 270)
-		(effects
-			(font
