File: fpgacarrierboard.kicad_pcb (KiCad board)
At the start: 6 copper layers, 150 x 100 mm, 211 parts, among them J1 Conn_01x06, J2 Conn_Coaxial, J3 HR911130C, J4 SFPK-SL, J5 Conn_02x10_Odd_Even, SW1 SW_Push, SW2 SW_Push, SW3 SW_Push, U1 TPS62130A, U2 TPS62130A, U3 TPS62130A, U4 TPS62130A, U5 TPS2592xx, U6 XC7A35T-FGG484, U7 W25Q128JVS, U8 RTL8211E-VB-CG, Y1 OT322550MJBA4SL, Y3 OT322525MJBA4SL

Commit message: Move signals off GND planes where they fit, stitch cut-off GND pieces
- In1.Cu: move 16 nets (62 segments) to In2.Cu/B.Cu where they fit with
  no clashes; 213 segments remain on In1.Cu
- In4.Cu: move 7 nets (54 segments) to In3.Cu/In2.Cu/B.Cu; BTN0, BTN1,
  1V0, 1V8, PHY_AVDD10 remain on In4.Cu
- Add GND stitching vias in cut-off In1.Cu, In4.Cu and B.Cu pieces
- Remove redundant SFP_VCCT via
- Known issue: C81, C83, C84 GND pads sit in B.Cu islands with no via
Routing:
- net SFP_VCCT: vias 4 -> 3
- net GND: vias 92 -> 109
